File: TD4.sch (KiCad schematic (older format))
At the start: 31 parts, among them J1 InPut, J2 DC_Jack, J3 OutPut, SW21 PWR_SW, U1 74HC74, U10 74HC283, U2 74HC10, U3 74HC161, U4 74HC161, U5 74HC161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

Commit message: 修正コミット
Parts:
- removed J1: InPut, Connector_PinHeader_2.54mm:PinHeader_1x05_P2.54mm_Vertical, symbol Connector_Generic:Conn_01x05
- removed RN1: 1K, Resistor_THT:R_Array_SIP9, symbol Device:R_Network08_Split
- added J1: InPut, Connector_PinHeader_2.54mm:PinHeader_1x06_P2.54mm_Vertical, symbol Connector_Generic:Conn_01x06
- added RN1: 1k, Resistor_THT:R_Array_SIP5, symbol Device:R_Network04
- J2: footprint shigobuFootPrint:18742DCjac -> Connector_BarrelJack:BarrelJack_Wuerth_6941xx301002
Connections:
- net +5V: now also J1.5 (Pin_5)
- net GND: now also J1.6 (Pin_6), RN1.1 (common)
- net ROM_D6: now also U2.9
- net ROM_D7: no longer U2.9
- net at U8.12 (I2b): now also J1.2 (Pin_2)
- net at U8.4 (I2a): now also J1.1 (Pin_1)
- net at U9.12 (I2b): now also J1.4 (Pin_4)
- net at U9.4 (I2a): now also J1.3 (Pin_3)
- net at D4.1 (K): now also RN1.5 (R4)
- net at D3.1 (K): now also RN1.4 (R3)
- net at D2.1 (K): now also RN1.3 (R2)
- net at D1.1 (K): now also RN1.2 (R1)
Other:
- moved on the sheet: C8, C9, U8, U9
