File: TD4.kicad_pcb (KiCad board)
At the start: 2 copper layers, 130 x 145 mm, 232 parts, among them J1 InPut, J2 DC_Jack, J3 OutPut, J4 Clock_Input, SW1 DIPSW, SW10 DIPSW, SW11 DIPSW, SW12 DIPSW, SW13 DIPSW, SW14 DIPSW, SW15 DIPSW, SW16 DIPSW, SW17 Manual Clock, SW18 Reset, SW19 FSW, SW2 DIPSW, SW20 SW_Rotary2x4, SW21 PWR_SW, SW3 DIPSW, SW4 DIPSW, SW5 DIPSW, SW6 DIPSW, SW7 DIPSW, SW8 DIPSW, SW9 DIPSW, U1 74HC74, U10 74HC283, U11 74HC138, U12 74HC540, U13 74HC14, U14 74HC138, U2 74HC10, U3 74HC161, U4 74HC161, U5 74HC161, U6 74HC161, U7 74HC32, U8 74HC153, U9 74HC153

Commit message: 修正コミット
Parts:
- removed R12, R14: 100, Resistor_THT:R_Axial_DIN0207_L6.3mm_D2.5mm_P7.62mm_Horizontal
- J1: footprint Connector_PinHeader_2.54mm:PinHeader_1x05_P2.54mm_Vertical -> Connector_PinHeader_2.54mm:PinHeader_1x06_P2.54mm_Vertical
- J2: footprint shigobuFootPrint:18742DCjac -> Connector_BarrelJack:BarrelJack_Wuerth_6941xx301002
- RN1: value 1K -> 1k; footprint Resistor_THT:R_Array_SIP9 -> Resistor_THT:R_Array_SIP5
- SW17, SW18: footprint Button_Switch_THT:SW_Tactile_Straight_KSA0Axx1LFTR -> Button_Switch_THT:SW_TH_Tactile_Omron_B3F-10xx
- moved RN1 27.3 mm to (144.9, 47.9), turned to 180 degrees
- moved R11 27.3 mm to (42.1, 64.4), turned to 0 degrees
- moved R15 25.9 mm to (49.8, 69.3), turned to 180 degrees
- moved J2 13.6 mm to (43.7, 80.7), turned to 270 degrees
- moved sym2 7.62 mm to (43.2, 73.3)
- moved D149 4.06 mm to (61.4, 42.8)
- moved D150 4.06 mm to (61.4, 47.9)
- moved D151 4.06 mm to (61.4, 53.0)
- moved D152 4.06 mm to (61.4, 58.1)
- moved C10 2.59 mm to (43.8, 89.8)
- moved SW20 1.52 mm to (46.1, 50.5)
- moved SW17 1.12 mm to (123.2, 171.1)
Connections:
- R11 pad 1: Net-(R11-Pad1) -> CLOCK
- RN1 pad 2: Net-(J1-Pad4) -> Net-(D1-Pad1)
- RN1 pad 3: Net-(J1-Pad3) -> Net-(D2-Pad1)
- RN1 pad 4: Net-(J1-Pad2) -> Net-(D3-Pad1)
- RN1 pad 5: Net-(J1-Pad1) -> Net-(D4-Pad1)
- SW17 pad 2: Net-(R2-Pad2) -> GND
- SW18 pad 2: Net-(R3-Pad2) -> GND
- SW20 pad 1: CLOCK -> Net-(R11-Pad2)
- SW20 pad 2: Net-(R12-Pad1) -> Net-(C14-Pad1)
- SW20 pad 3: Net-(R11-Pad1) -> Net-(SW20-Pad3)
- SW20 pad 4: Net-(R14-Pad1) -> Net-(J4-Pad3)
- U13 pad 2: Net-(R11-Pad2) -> Net-(SW20-Pad3)
- U2 pad 9: ROM_D7 -> ROM_D6
Routing:
- net GND: track 553.1 -> 1.81 mm, vias 0 -> 6
- net Net-(R10-Pad2): track 129.0 -> 226.2 mm
- net Net-(C14-Pad2): track 133.3 -> 169.0 mm
- net /L4: track 138.9 -> 110.2 mm, vias 0 -> 1
- net Net-(R3-Pad2): track 170.4 -> 143.8 mm
- net Net-(R11-Pad1): track 24.9 -> 0.00 mm
- net ROM_D6: track 47.8 -> 72.5 mm
- net Net-(D102-Pad1): track 69.0 -> 93.4 mm
- net CLOCK: track 180.2 -> 157.3 mm, vias 0 -> 1
- net /L3: track 50.6 -> 72.8 mm
- net Net-(J1-Pad4): track 48.8 -> 26.8 mm
- net /L2: track 74.4 -> 52.5 mm, vias 0 -> 1
- net Net-(J1-Pad3): track 58.0 -> 36.2 mm
- net ROM_D2: track 71.7 -> 93.1 mm
- net Net-(R2-Pad2): track 186.6 -> 206.5 mm
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Other:
- board text added: "5V"
- board text added: "TD4 shigobu V2"
- board text removed: "TD4 shigobu"

Commit message: 配線やり直し
Routing:
- net /ROM/540-3: track 310.7 -> 309.7 mm
- net /ROM/540-4: track 310.6 -> 309.8 mm
- net /ROM/540-2: track 313.2 -> 312.5 mm
- net /ROM/540-0: track 310.2 -> 310.8 mm
